Commit message: Centering the Chasis done

File: description/robot.xacro (robot description, xacro)
@@ -40,5 +40,5 @@
         </inertial>
         <visual name="">
-            <origin xyz="0.0 0.02 0.0" rpy="0.0 0.0 -1.5708"/>
+            <origin xyz="0.0 0.0115 0.0" rpy="0.0 0.0 -1.5708"/>
             <geometry>
                 <mesh filename="file://$(find rover)/description/stl/Chasis.stl" scale="0.01 0.01 0.01"/>/>

Commit message: Wheels added, must be moved to the right postion

File: description/robot.xacro (robot description, xacro)
@@ -1,6 +1,7 @@
 <?xml version="1.0"?>
 <robot xmlns:xacro="http://www.ros.org/wiki/xacro"  name="robot">
-    <!-- Example link -->
+    <!--Joint Definition-->
     <link name="base_link"></link>
+    <!--Chasis Definition-->
     <joint name="base_joint" type="fixed">
         <origin xyz="0.0 0.0 0.0" rpy="0.0 0.0 0.0"/>
@@ -33,4 +34,30 @@
         <axis xyz="0.0 0.0 0.0" />
     </joint>
+    <!--Wheel Joints Definition-->
+    <joint name="wheel_left_front_joint" type="fixed">
+        <origin xyz="0.0 0.0 0.0" rpy="3.14 -1.5708 0.0"/>
+        <parent link="arm_left_front_link"/>
+        <child link="wheel_left_front_link"/>
+        <axis xyz="0.0 0.0 0.0"/>
+    </joint>
+    <joint name="wheel_left_back_joint" type="fixed">
+        <origin xyz="0.0 0.0 0.0" rpy="3.14 -1.5708 0.0"/>
+        <parent link="arm_left_back_link"/>
+        <child link="wheel_left_back_link"/>
+        <axis xyz="0.0 0.0 0.0"/>
+    </joint>
+    <joint name="wheel_right_front_joint" type="fixed">
+        <origin xyz="0.0 0.0 0.0" rpy="3.14 -1.5708 0.0"/>
+        <parent link="arm_right_front_link"/>
+        <child link="wheel_right_front_link"/>
+        <axis xyz="0.0 0.0 0.0"/>
+    </joint>
+    <joint name="wheel_back_front_joint" type="fixed">
+        <origin xyz="0.0 0.0 0.0" rpy="3.14 -1.5708 0.0"/>
+        <parent link="arm_right_back_link"/>
+        <child link="wheel_right_back_link"/>
+        <axis xyz="0.0 0.0 0.0"/>
+    </joint>
+    <!--Link Definition-->
     <link name="chasis_link">
         <inertial>
@@ -147,3 +174,96 @@
         </collision>
     </link>
+    <!--Wheel Link Definition-->
+    <link name="wheel_left_front_link">
+        <inertial>
+            <origin xyz="0.0 0.0 0.0" rpy="0.0 0.0 0.0"/>
+            <mass value="0.0"/>
+            <inertia ixx="0.0" ixy="0.0" ixz="0.0" iyy="0.0" iyz="0.0" izz="0.0"/>
+        </inertial>
+        <visual name="">
+            <origin xyz="0.0 0.0 0.0" rpy="0.0 0.0 0.0"/>
+            <geometry>
+                <cylinder radius="0.07" length="0.05"/>
+            </geometry>
+            <material name="">
+                <color rgba="1.0 0.0 0.0 1.0"/>
+                <texture filename=""/>
+            </material>
+        </visual>
+        <collision>
+            <origin xyz="0.0 0.0 0.0" rpy="0.0 0.0 0.0"/>
+            <geometry>
+                <cylinder radius="0.07" length="0.05"/>
+            </geometry>
+        </collision>
+    </link>
+    <link name="wheel_left_back_link">
+        <inertial>
+            <origin xyz="0.0 0.0 0.0" rpy="0.0 0.0 0.0"/>
+            <mass value="0.0"/>
+            <inertia ixx="0.0" ixy="0.0" ixz="0.0" iyy="0.0" iyz="0.0" izz="0.0"/>
+        </inertial>
+        <visual name="">
+            <origin xyz="0.0 0.0 0.0" rpy="0.0 0.0 0.0"/>
+            <geometry>
+                <cylinder radius="0.07" length="0.05"/>
+            </geometry>
+            <material name="">
+                <color rgba="1.0 0.0 0.0 1.0"/>
+                <texture filename=""/>
+            </material>
+        </visual>
+        <collision>
+            <origin xyz="0.0 0.0 0.0" rpy="0.0 0.0 0.0"/>
+            <geometry>
+                <cylinder radius="0.07" length="0.05"/>
+            </geometry>
+        </collision>
+    </link>
+    <link name="wheel_right_front_link">
+        <inertial>
+            <origin xyz="0.0 0.0 0.0" rpy="0.0 0.0 0.0"/>
+            <mass value="0.0"/>
+            <inertia ixx="0.0" ixy="0.0" ixz="0.0" iyy="0.0" iyz="0.0" izz="0.0"/>
+        </inertial>
+        <visual name="">
+            <origin xyz="0.0 0.0 0.0" rpy="0.0 0.0 0.0"/>
+            <geometry>
+                <cylinder radius="0.07" length="0.05"/>
+            </geometry>
+            <material name="">
+                <color rgba="1.0 0.0 0.0 1.0"/>
+                <texture filename=""/>
+            </material>
+        </visual>
+        <collision>
+            <origin xyz="0.0 0.0 0.0" rpy="0.0 0.0 0.0"/>
+            <geometry>
+                <cylinder radius="0.07" length="0.05"/>
+            </geometry>
+        </collision>
+    </link>
+    <link name="wheel_right_back_link">
+        <inertial>
+            <origin xyz="0.0 0.0 0.0" rpy="0.0 0.0 0.0"/>
+            <mass value="0.0"/>
+            <inertia ixx="0.0" ixy="0.0" ixz="0.0" iyy="0.0" iyz="0.0" izz="0.0"/>
+        </inertial>
+        <visual name="">
+            <origin xyz="0.0 0.0 0.0" rpy="0.0 0.0 0.0"/>
+            <geometry>
+                <cylinder radius="0.07" length="0.05"/>
+            </geometry>
+            <material name="">
+                <color rgba="1.0 0.0 0.0 1.0"/>
+                <texture filename=""/>
+            </material>
+        </visual>
+        <collision>
+            <origin xyz="0.0 0.0 0.0" rpy="0.0 0.0 0.0"/>
+            <geometry>
+                <cylinder radius="0.07" length="0.05"/>
+            </geometry>
+        </collision>
+    </link>
 </robot>

Commit message: Wheel are on right pos

File: description/robot.xacro (robot description, xacro)
@@ -1,4 +1,7 @@
 <?xml version="1.0"?>
 <robot xmlns:xacro="http://www.ros.org/wiki/xacro"  name="robot">
+    <!--Defines-->
+    <xacro:property name="length_wheel" value="0.04"/>
+    <xacro:property name="radius_wheel" value="0.07"/>
     <!--Joint Definition-->
     <link name="base_link"></link>
@@ -36,5 +39,5 @@
     <!--Wheel Joints Definition-->
     <joint name="wheel_left_front_joint" type="fixed">
-        <origin xyz="0.0 0.0 0.0" rpy="3.14 -1.5708 0.0"/>
+        <origin xyz="${0.03+length_wheel/2} -0.067 -0.04 " rpy="3.14 -1.5708 0.0"/>
         <parent link="arm_left_front_link"/>
         <child link="wheel_left_front_link"/>
@@ -42,5 +45,5 @@
     </joint>
     <joint name="wheel_left_back_joint" type="fixed">
-        <origin xyz="0.0 0.0 0.0" rpy="3.14 -1.5708 0.0"/>
+        <origin xyz="${0.03+length_wheel/2} -0.067 0.04 " rpy="3.14 -1.5708 0.0"/>
         <parent link="arm_left_back_link"/>
         <child link="wheel_left_back_link"/>
@@ -48,5 +51,5 @@
     </joint>
     <joint name="wheel_right_front_joint" type="fixed">
-        <origin xyz="0.0 0.0 0.0" rpy="3.14 -1.5708 0.0"/>
+        <origin xyz="${0.03+length_wheel/2} -0.067 0.04 " rpy="3.14 -1.5708 0.0"/>
         <parent link="arm_right_front_link"/>
         <child link="wheel_right_front_link"/>
@@ -54,5 +57,5 @@
     </joint>
     <joint name="wheel_back_front_joint" type="fixed">
-        <origin xyz="0.0 0.0 0.0" rpy="3.14 -1.5708 0.0"/>
+        <origin xyz="${0.03+length_wheel/2} -0.067 -0.04 " rpy="3.14 -1.5708 0.0"/>
         <parent link="arm_right_back_link"/>
         <child link="wheel_right_back_link"/>
@@ -184,15 +187,15 @@
             <origin xyz="0.0 0.0 0.0" rpy="0.0 0.0 0.0"/>
             <geometry>
-                <cylinder radius="0.07" length="0.05"/>
-            </geometry>
-            <material name="">
-                <color rgba="1.0 0.0 0.0 1.0"/>
-                <texture filename=""/>
-            </material>
-        </visual>
-        <collision>
-            <origin xyz="0.0 0.0 0.0" rpy="0.0 0.0 0.0"/>
-            <geometry>
-                <cylinder radius="0.07" length="0.05"/>
+                 <cylinder radius="${radius_wheel}" length="${length_wheel}"/>
+            </geometry>
+            <material name="">
+                <color rgba="1.0 0.0 0.0 1.0"/>
+                <texture filename=""/>
+            </material>
+        </visual>
+        <collision>
+            <origin xyz="0.0 0.0 0.0" rpy="0.0 0.0 0.0"/>
+            <geometry>
+                 <cylinder radius="${radius_wheel}" length="${length_wheel}"/>
             </geometry>
         </collision>
@@ -207,15 +210,15 @@
             <origin xyz="0.0 0.0 0.0" rpy="0.0 0.0 0.0"/>
             <geometry>
-                <cylinder radius="0.07" length="0.05"/>
-            </geometry>
-            <material name="">
-                <color rgba="1.0 0.0 0.0 1.0"/>
-                <texture filename=""/>
-            </material>
-        </visual>
-        <collision>
-            <origin xyz="0.0 0.0 0.0" rpy="0.0 0.0 0.0"/>
-            <geometry>
-                <cylinder radius="0.07" length="0.05"/>
+                  <cylinder radius="${radius_wheel}" length="${length_wheel}"/>
+            </geometry>
+            <material name="">
+                <color rgba="1.0 0.0 0.0 1.0"/>
+                <texture filename=""/>
+            </material>
+        </visual>
+        <collision>
+            <origin xyz="0.0 0.0 0.0" rpy="0.0 0.0 0.0"/>
+            <geometry>
+                  <cylinder radius="${radius_wheel}" length="${length_wheel}"/>
             </geometry>
         </collision>
@@ -230,15 +233,15 @@
             <origin xyz="0.0 0.0 0.0" rpy="0.0 0.0 0.0"/>
             <geometry>
-                <cylinder radius="0.07" length="0.05"/>
-            </geometry>
-            <material name="">
-                <color rgba="1.0 0.0 0.0 1.0"/>
-                <texture filename=""/>
-            </material>
-        </visual>
-        <collision>
-            <origin xyz="0.0 0.0 0.0" rpy="0.0 0.0 0.0"/>
-            <geometry>
-                <cylinder radius="0.07" length="0.05"/>
+                 <cylinder radius="${radius_wheel}" length="${length_wheel}"/>
+            </geometry>
+            <material name="">
+                <color rgba="1.0 0.0 0.0 1.0"/>
+                <texture filename=""/>
+            </material>
+        </visual>
+        <collision>
+            <origin xyz="0.0 0.0 0.0" rpy="0.0 0.0 0.0"/>
+            <geometry>
+                 <cylinder radius="${radius_wheel}" length="${length_wheel}"/>
             </geometry>
         </collision>
@@ -253,15 +256,15 @@
             <origin xyz="0.0 0.0 0.0" rpy="0.0 0.0 0.0"/>
             <geometry>
-                <cylinder radius="0.07" length="0.05"/>
-            </geometry>
-            <material name="">
-                <color rgba="1.0 0.0 0.0 1.0"/>
-                <texture filename=""/>
-            </material>
-        </visual>
-        <collision>
-            <origin xyz="0.0 0.0 0.0" rpy="0.0 0.0 0.0"/>
-            <geometry>
-                <cylinder radius="0.07" length="0.05"/>
+                <cylinder radius="${radius_wheel}" length="${length_wheel}"/>
+            </geometry>
+            <material name="">
+                <color rgba="1.0 0.0 0.0 1.0"/>
+                <texture filename=""/>
+            </material>
+        </visual>
+        <collision>
+            <origin xyz="0.0 0.0 0.0" rpy="0.0 0.0 0.0"/>
+            <geometry>
+                <cylinder radius="${radius_wheel}" length="${length_wheel}"/>
             </geometry>
         </collision>

Commit message: Wheels are shown and working in rviz2 added joint state

File: description/robot.xacro (robot description, xacro)
@@ -11,5 +11,4 @@
         <parent link="base_link"/>
         <child link="chasis_link"/>
-        <axis xyz="0.0 0.0 0.0"/>
     </joint>
     <joint name="arm_left_front_joint" type="fixed">
@@ -17,5 +16,4 @@
         <parent link="chasis_link"/>
         <child link="arm_left_front_link"/>
-        <axis xyz="0.0 0.0 0.0" />
     </joint>
     <joint name="arm_left_back_joint" type="fixed">
@@ -23,5 +21,4 @@
         <parent link="chasis_link"/>
         <child link="arm_left_back_link"/>
-        <axis xyz="0.0 0.0 0.0" />
     </joint>
     <joint name="arm_right_front_joint" type="fixed">
@@ -29,5 +26,4 @@
         <parent link="chasis_link"/>
         <child link="arm_right_front_link"/>
-        <axis xyz="0.0 0.0 0.0" />
     </joint>
     <joint name="arm_right_back_joint" type="fixed">
@@ -35,30 +31,29 @@
         <parent link="chasis_link"/>
         <child link="arm_right_back_link"/>
-        <axis xyz="0.0 0.0 0.0" />
     </joint>
     <!--Wheel Joints Definition-->
-    <joint name="wheel_left_front_joint" type="fixed">
+    <joint name="wheel_left_front_joint" type="continuous">
         <origin xyz="${0.03+length_wheel/2} -0.067 -0.04 " rpy="3.14 -1.5708 0.0"/>
         <parent link="arm_left_front_link"/>
         <child link="wheel_left_front_link"/>
-        <axis xyz="0.0 0.0 0.0"/>
-    </joint>
-    <joint name="wheel_left_back_joint" type="fixed">
+        <axis xyz="0.0 0.0 1.0"/>
+    </joint>
+    <joint name="wheel_left_back_joint" type="continuous">
         <origin xyz="${0.03+length_wheel/2} -0.067 0.04 " rpy="3.14 -1.5708 0.0"/>
         <parent link="arm_left_back_link"/>
         <child link="wheel_left_back_link"/>
-        <axis xyz="0.0 0.0 0.0"/>
-    </joint>
-    <joint name="wheel_right_front_joint" type="fixed">
+        <axis xyz="0.0 0.0 1.0"/>
+    </joint>
+    <joint name="wheel_right_front_joint" type="continuous">
         <origin xyz="${0.03+length_wheel/2} -0.067 0.04 " rpy="3.14 -1.5708 0.0"/>
         <parent link="arm_right_front_link"/>
         <child link="wheel_right_front_link"/>
-        <axis xyz="0.0 0.0 0.0"/>
-    </joint>
-    <joint name="wheel_back_front_joint" type="fixed">
+        <axis xyz="0.0 0.0 1.0"/>
+    </joint>
+    <joint name="wheel_back_front_joint" type="continuous">
         <origin xyz="${0.03+length_wheel/2} -0.067 -0.04 " rpy="3.14 -1.5708 0.0"/>
         <parent link="arm_right_back_link"/>
         <child link="wheel_right_back_link"/>
-        <axis xyz="0.0 0.0 0.0"/>
+        <axis xyz="0.0 0.0 1.0"/>
     </joint>
     <!--Link Definition-->
@@ -67,5 +62,5 @@
             <origin xyz="0.0 0.0 0.0" rpy="0.0 0.0 0.0"/>
             <mass value="20.0"/>
-            <inertia ixx="0.0" ixy="0.0" ixz="0.0" iyy="0.0" iyz="0.0" izz="0.0"/>
+            <inertia ixx="${0.3}" ixy="0.0" ixz="0.0" iyy="0.0" iyz="0.0" izz="0.0"/>
         </inertial>
         <visual name="">
@@ -89,5 +84,5 @@
             <origin xyz="0.0 0.0 0.0" rpy="0.0 0.0 0.0"/>
             <mass value="0.0"/>
-            <inertia ixx="0.0" ixy="0.0" ixz="0.0" iyy="0.0" iyz="0.0" izz="0.0"/>
+            <inertia ixx="0.010653" ixy=" 0.001298" ixz="-0.000756" iyy="-0.000756" iyz="-0.000756" izz="-0.000756"/>
         </inertial>
         <visual name="">
@@ -112,5 +107,5 @@
             <origin xyz="0.0 0.0 0.0" rpy="0.0 0.0 0.0"/>
             <mass value="0.0"/>
-            <inertia ixx="0.0" ixy="0.0" ixz="0.0" iyy="0.0" iyz="0.0" izz="0.0"/>
+             <inertia ixx="0.010653" ixy=" 0.001298" ixz="-0.000756" iyy="-0.000756" iyz="-0.000756" izz="-0.000756"/>
         </inertial>
         <visual name="">
@@ -135,5 +130,5 @@
             <origin xyz="0.0 0.0 0.0" rpy="0.0 0.0 0.0"/>
             <mass value="0.0"/>
-            <inertia ixx="0.0" ixy="0.0" ixz="0.0" iyy="0.0" iyz="0.0" izz="0.0"/>
+            <inertia ixx="0.010653" ixy=" 0.001298" ixz="-0.000756" iyy="-0.000756" iyz="-0.000756" izz="-0.000756"/>
         </inertial>
         <visual name="">
@@ -158,5 +153,5 @@
             <origin xyz="0.0 0.0 0.0" rpy="0.0 0.0 0.0"/>
             <mass value="0.0"/>
-            <inertia ixx="0.0" ixy="0.0" ixz="0.0" iyy="0.0" iyz="0.0" izz="0.0"/>
+            <inertia ixx="0.010653" ixy=" 0.001298" ixz="-0.000756" iyy="-0.000756" iyz="-0.000756" izz="-0.000756"/>
         </inertial>
         <visual name="">
