Commit message: Wheel seperate in new File

File: description/robot.urdf.xacro (robot description, xacro)
@@ -1,5 +1,4 @@
 <?xml version="1.0"?>
 <robot xmlns:xacro="http://www.ros.org/wiki/xacro"  name="robot">
-    <!-- Example link -->
     <xacro:include filename="robot.xacro"/>
 </robot>

File: description/robot.xacro (robot description, xacro)
@@ -1,7 +1,6 @@
 <?xml version="1.0"?>
 <robot xmlns:xacro="http://www.ros.org/wiki/xacro"  name="robot">
+    <xacro:include filename="wheel.xacro"/>
     <!--Defines-->
-    <xacro:property name="length_wheel" value="0.04"/>
-    <xacro:property name="radius_wheel" value="0.07"/>
     <!--Joint Definition-->
     <link name="base_link"></link>
@@ -173,95 +172,7 @@
     </link>
     <!--Wheel Link Definition-->
-    <link name="wheel_left_front_link">
-        <inertial>
-            <origin xyz="0.0 0.0 0.0" rpy="0.0 0.0 0.0"/>
-            <mass value="0.0"/>
-            <inertia ixx="0.0" ixy="0.0" ixz="0.0" iyy="0.0" iyz="0.0" izz="0.0"/>
-        </inertial>
-        <visual name="">
-            <origin xyz="0.0 0.0 0.0" rpy="0.0 0.0 0.0"/>
-            <geometry>
-                 <cylinder radius="${radius_wheel}" length="${length_wheel}"/>
-            </geometry>
-            <material name="">
-                <color rgba="1.0 0.0 0.0 1.0"/>
-                <texture filename=""/>
-            </material>
-        </visual>
-        <collision>
-            <origin xyz="0.0 0.0 0.0" rpy="0.0 0.0 0.0"/>
-            <geometry>
-                 <cylinder radius="${radius_wheel}" length="${length_wheel}"/>
-            </geometry>
-        </collision>
-    </link>
-    <link name="wheel_left_back_link">
-        <inertial>
-            <origin xyz="0.0 0.0 0.0" rpy="0.0 0.0 0.0"/>
-            <mass value="0.0"/>
-            <inertia ixx="0.0" ixy="0.0" ixz="0.0" iyy="0.0" iyz="0.0" izz="0.0"/>
-        </inertial>
-        <visual name="">
-            <origin xyz="0.0 0.0 0.0" rpy="0.0 0.0 0.0"/>
-            <geometry>
-                  <cylinder radius="${radius_wheel}" length="${length_wheel}"/>
-            </geometry>
-            <material name="">
-                <color rgba="1.0 0.0 0.0 1.0"/>
-                <texture filename=""/>
-            </material>
-        </visual>
-        <collision>
-            <origin xyz="0.0 0.0 0.0" rpy="0.0 0.0 0.0"/>
-            <geometry>
-                  <cylinder radius="${radius_wheel}" length="${length_wheel}"/>
-            </geometry>
-        </collision>
-    </link>
-    <link name="wheel_right_front_link">
-        <inertial>
-            <origin xyz="0.0 0.0 0.0" rpy="0.0 0.0 0.0"/>
-            <mass value="0.0"/>
-            <inertia ixx="0.0" ixy="0.0" ixz="0.0" iyy="0.0" iyz="0.0" izz="0.0"/>
-        </inertial>
-        <visual name="">
-            <origin xyz="0.0 0.0 0.0" rpy="0.0 0.0 0.0"/>
-            <geometry>
-                 <cylinder radius="${radius_wheel}" length="${length_wheel}"/>
-            </geometry>
-            <material name="">
-                <color rgba="1.0 0.0 0.0 1.0"/>
-                <texture filename=""/>
-            </material>
-        </visual>
-        <collision>
-            <origin xyz="0.0 0.0 0.0" rpy="0.0 0.0 0.0"/>
-            <geometry>
-                 <cylinder radius="${radius_wheel}" length="${length_wheel}"/>
-            </geometry>
-        </collision>
-    </link>
-    <link name="wheel_right_back_link">
-        <inertial>
-            <origin xyz="0.0 0.0 0.0" rpy="0.0 0.0 0.0"/>
-            <mass value="0.0"/>
-            <inertia ixx="0.0" ixy="0.0" ixz="0.0" iyy="0.0" iyz="0.0" izz="0.0"/>
-        </inertial>
-        <visual name="">
-            <origin xyz="0.0 0.0 0.0" rpy="0.0 0.0 0.0"/>
-            <geometry>
-                <cylinder radius="${radius_wheel}" length="${length_wheel}"/>
-            </geometry>
-            <material name="">
-                <color rgba="1.0 0.0 0.0 1.0"/>
-                <texture filename=""/>
-            </material>
-        </visual>
-        <collision>
-            <origin xyz="0.0 0.0 0.0" rpy="0.0 0.0 0.0"/>
-            <geometry>
-                <cylinder radius="${radius_wheel}" length="${length_wheel}"/>
-            </geometry>
-        </collision>
-    </link>
+    <xacro:wheel side="left" front="front"/>
+    <xacro:wheel side="left" front="back"/>
+    <xacro:wheel side="right" front="front"/>
+    <xacro:wheel side="right" front="back"/>
 </robot>

Commit message: Drive Plugin added
Added Drive plugin for Rover. Renamed Launch Script Typo and added Base link

File: description/robot.urdf.xacro (robot description, xacro)
@@ -2,3 +2,4 @@
 <robot xmlns:xacro="http://www.ros.org/wiki/xacro"  name="robot">
     <xacro:include filename="robot.xacro"/>
-</robot>
+    <xacro:include filename="gazebo.xacro"/>
+    </robot>

File: description/robot.xacro (robot description, xacro)
@@ -6,4 +6,6 @@
     <xacro:property name="radius_wheel" value="0.07"/>
     <xacro:property name="mass_wheel" value="1"/>
+    <link name="base_link">
+    </link>
     <!--Defines-->
     <!--Wheel Link Definition-->
@@ -43,5 +45,5 @@
                 </geometry>
             </collision>
-        </link>
+    </link>
     <link name="wheel_right_front_link">
             <xacro:inertial_cylinder mass="1" length="0.04" radius="0.07">
@@ -93,5 +95,5 @@
         </visual>
         <collision>
-            <origin xyz="0.0 0.0 0.1" rpy="0.0 0.0 0.0"/>
+            <origin xyz="0.0 0.0 0.2" rpy="0.0 0.0 0.0"/>
             <geometry>
                 <box size="0.6 0.3 0.2"/>
@@ -113,5 +115,5 @@
             <origin xyz="0.0 0.0 0.0" rpy="0.0 0.0 0.0"/>
             <geometry>
-                <box size="0.5 0.2 0.1"/>
+                <box size="0.2 0.2 0.1"/>
             </geometry>
         </collision>
@@ -131,5 +133,5 @@
             <origin xyz="0.0 0.0 0.0" rpy="0.0 0.0 0.0"/>
             <geometry>
-                <box size="0.5 0.2 0.1"/>
+                <box size="0.2 0.2 0.1"/>
             </geometry>
         </collision>
@@ -149,5 +151,5 @@
             <origin xyz="0.0 0.0 0.0" rpy="0.0 0.0 0.0"/>
             <geometry>
-                <box size="0.5 0.2 0.1"/>
+                <box size="0.2 0.2 0.1"/>
             </geometry>
         </collision>
@@ -167,9 +169,14 @@
             <origin xyz="0.0 0.0 0.0" rpy="0.0 0.0 0.0"/>
             <geometry>
-                <box size="0.5 0.2 0.1"/>
+                <box size="0.2 0.2 0.1"/>
             </geometry>
         </collision>
     </link>
      <!--Chasis Definition-->
+    <joint name="base_joint" type="fixed">
+        <origin xyz="0.0 0.0 0.1" rpy="0.0 0.0 0.0"/>
+        <parent link="base_link"/>
+        <child link="chasis_link"/>
+        </joint>
     <joint name="arm_left_front_joint" type="fixed">
         <origin xyz="-0.15 -0.0955 0.1" rpy="0.0 0.0 -1.5708"/>
@@ -211,5 +218,5 @@
         <axis xyz="0.0 0.0 1.0"/>
     </joint>
-    <joint name="wheel_back_front_joint" type="continuous">
+    <joint name="wheel_right_back_joint" type="continuous">
         <origin xyz="${0.03+length_wheel/2} -0.067 -0.04 " rpy="3.14 -1.5708 0.0"/>
         <parent link="arm_right_back_link"/>
