Commit message: Added Lidar

File: description/color.xacro (robot description, xacro)
@@ -1,4 +1,4 @@
 <?xml version="1.0"?>
-<robot xmlns:xacro="http://www.ros.org/wiki/xacro"  name="robot">
+<robot xmlns:xacro="http://www.ros.org/wiki/xacro"  name="rover">
     <material name="white">
         <color rgba="1 1 1 1"/>

File: description/robot.urdf.xacro (robot description, xacro)
@@ -3,3 +3,4 @@
     <xacro:include filename="robot.xacro"/>
     <xacro:include filename="gazebo.xacro"/>
+    <xacro:include filename="lidar.xacro"/>
     </robot>

File: description/robot.xacro (robot description, xacro)
@@ -95,7 +95,7 @@
         </visual>
         <collision>
-            <origin xyz="0.0 0.0 0.1" rpy="0.0 0.0 0.0"/>
-            <geometry>
-                <box size="0.6 0.2 0.2"/>
+            <origin xyz="0.0 0.0 0" rpy="0.0 0.0 0.0"/>
+            <geometry>
+                <box size="0.6 0.2 0.01"/>
             </geometry>
         </collision>
