Commit message: Added Lidar Sensor and SLAM config

File: description/lidar.xacro (robot description, xacro)
@@ -7,5 +7,5 @@
     </joint>
     <link name="laser_frame">
-        <xacro:inertial_cylinder mass="0.1" length="0.0" radius="0.0">
+        <xacro:inertial_cylinder mass="0.1" length="0.0"  radius="0.025">
             <origin xyz="0.0 0.0 0.0" rpy="0.0 0.0 0.0"/>
         </xacro:inertial_cylinder>
@@ -39,5 +39,5 @@
                 <range>
                     <min>0.3</min>
-                    <max>4</max>
+                    <max>12</max>
                 </range>
             </ray>

File: description/robot.xacro (robot description, xacro)
@@ -8,4 +8,11 @@
     <link name="base_link">
     </link>
+    <link name="base_footprint">
+    </link>
+    <joint name="base_footprint_joint" type="fixed">
+        <parent link="base_link"/>
+        <child link="base_footprint"/>
+        <origin xyz="0 0 0" rpy="0 0 0"/>
+    </joint>
     <!--Defines-->
     <!--Wheel Link Definition-->
