Commit message: Renamned Bot and tweek parms for gazebo

File: description/gazebo.xacro (robot description, xacro)
@@ -1,12 +1,12 @@
 <?xml version="1.0"?>
-<robot xmlns:xacro="http://www.ros.org/wiki/xacro"  name="robot">
+<robot xmlns:xacro="http://www.ros.org/wiki/xacro"  name="rover">
         <gazebo>
-              <plugin name='skid_steer_drive' filename='libgazebo_ros_diff_drive.so'>
+          <plugin name='skid_steer_drive' filename='libgazebo_ros_diff_drive.so'>
         <ros>
           <!-- Set namespace -->
           <namespace>/</namespace>
           <!-- Remap default topics -->
-          <remapping>cmd_vel:=cmd_demo</remapping>
-          <remapping>odom:=odom_demo</remapping>
+          <remapping>cmd_vel:=cmd_vel</remapping>
+          <remapping>odom:=odom</remapping>
         </ros>
         <!-- Update rate -->
@@ -21,18 +21,54 @@
         <right_joint>wheel_right_back_joint</right_joint>
         <!-- kinematics -->
-        <wheel_separation>0.25</wheel_separation>
-        <wheel_separation>0.25</wheel_separation>
+        <wheel_separation>0.4</wheel_separation>
+        <wheel_separation>0.4</wheel_separation>
         <wheel_diameter>0.14</wheel_diameter>
         <wheel_diameter>0.14</wheel_diameter>
         <!-- limits -->
-        <max_wheel_torque>20</max_wheel_torque>
-        <max_wheel_acceleration>1.0</max_wheel_acceleration>
+        <max_wheel_torque>400</max_wheel_torque>
+        <max_wheel_acceleration>2.0</max_wheel_acceleration>
         <!-- output -->
         <publish_odom>true</publish_odom>
         <publish_odom_tf>true</publish_odom_tf>
         <publish_wheel_tf>true</publish_wheel_tf>
-        <odometry_frame>odom_demo</odometry_frame>
+        <odometry_frame>odom</odometry_frame>
         <robot_base_frame>base_link</robot_base_frame>
       </plugin>
     </gazebo>
+    <gazebo reference="wheel_left_front_link">
+      <mu1>20</mu1>
+      <mu2>10</mu2>
+      <minDepth>0.0001</minDepth>
+      <kp>100000000</kp>
+      <kd>100</kd>
+      <slip1>1.0</slip1>
+      <slip2>0.0</slip2>
+    </gazebo>
+     <gazebo reference="wheel_left_back_link">
+      <mu1>20</mu1>
+      <mu2>10</mu2>
+      <minDepth>0.0001</minDepth>
+      <kp>100000000</kp>
+      <kd>100</kd>
+      <slip1>1.0</slip1>
+      <slip2>0.0</slip2>
+    </gazebo>
+     <gazebo reference="wheel_right_front_link">
+      <mu1>20</mu1>
+      <mu2>10</mu2>
+      <minDepth>0.0001</minDepth>
+      <kp>100000000</kp>
+      <kd>100</kd>
+      <slip1>1.0</slip1>
+      <slip2>0.0</slip2>
+    </gazebo>
+     <gazebo reference="wheel_right_back_link">
+      <mu1>20</mu1>
+      <mu2>10</mu2>
+      <minDepth>0.0001</minDepth>
+      <kp>100000000</kp>
+      <kd>100</kd>
+      <slip1>1.0</slip1>
+      <slip2>0.0</slip2>
+    </gazebo>
 </robot>

File: description/robot.urdf.xacro (robot description, xacro)
@@ -1,4 +1,4 @@
 <?xml version="1.0"?>
-<robot xmlns:xacro="http://www.ros.org/wiki/xacro"  name="robot">
+<robot xmlns:xacro="http://www.ros.org/wiki/xacro"  name="rover">
     <xacro:include filename="robot.xacro"/>
     <xacro:include filename="gazebo.xacro"/>

File: description/robot.xacro (robot description, xacro)
@@ -1,4 +1,4 @@
 <?xml version="1.0"?>
-<robot xmlns:xacro="http://www.ros.org/wiki/xacro"  name="robot">
+<robot xmlns:xacro="http://www.ros.org/wiki/xacro"  name="rover">
     <xacro:include filename="intertia.xacro"/>
     <xacro:include filename="color.xacro"/>
@@ -84,9 +84,9 @@
     <!--Joint Definition-->
     <link name="chasis_link">
-        <xacro:inertial_box mass="10" x="0.6" y="0.3" z="0.2">
-            <oigin xyz="0.0 0 0.0" rpy="0 0 0"/>
+        <xacro:inertial_box mass="20" x="0.6" y="0.3" z="0.2">
+            <oigin xyz="0.0 0.0 0.0" rpy="0 0 0"/>
         </xacro:inertial_box>
         <visual>
-            <origin xyz="0.0 0.0115 0.0" rpy="0.0 0.0 -1.5708"/>
+            <origin xyz="0.0 0.0115 -0.1" rpy="0.0 0.0 -1.5708"/>
             <geometry>
                 <mesh filename="file://$(find rover)/description/stl/Chasis.stl" scale="0.01 0.01 0.01"/>
@@ -95,7 +95,7 @@
         </visual>
         <collision>
-            <origin xyz="0.0 0.0 0.2" rpy="0.0 0.0 0.0"/>
-            <geometry>
-                <box size="0.6 0.3 0.2"/>
+            <origin xyz="0.0 0.0 0.1" rpy="0.0 0.0 0.0"/>
+            <geometry>
+                <box size="0.6 0.2 0.2"/>
             </geometry>
         </collision>
@@ -115,5 +115,5 @@
             <origin xyz="0.0 0.0 0.0" rpy="0.0 0.0 0.0"/>
             <geometry>
-                <box size="0.2 0.2 0.1"/>
+                <box size="0.02 0.02 0.01"/>
             </geometry>
         </collision>
@@ -133,5 +133,5 @@
             <origin xyz="0.0 0.0 0.0" rpy="0.0 0.0 0.0"/>
             <geometry>
-                <box size="0.2 0.2 0.1"/>
+                <box size="0.02 0.02 0.01"/>
             </geometry>
         </collision>
@@ -150,6 +150,6 @@
         <collision>
             <origin xyz="0.0 0.0 0.0" rpy="0.0 0.0 0.0"/>
-            <geometry>
-                <box size="0.2 0.2 0.1"/>
+           <geometry>
+                <box size="0.02 0.02 0.01"/>
             </geometry>
         </collision>
@@ -169,5 +169,5 @@
             <origin xyz="0.0 0.0 0.0" rpy="0.0 0.0 0.0"/>
             <geometry>
-                <box size="0.2 0.2 0.1"/>
+                <box size="0.02 0.02 0.01"/>
             </geometry>
         </collision>
@@ -175,25 +175,25 @@
      <!--Chasis Definition-->
     <joint name="base_joint" type="fixed">
-        <origin xyz="0.0 0.0 0.1" rpy="0.0 0.0 0.0"/>
+        <origin xyz="0.0 0.0 0.2" rpy="0.0 0.0 0.0"/>
         <parent link="base_link"/>
         <child link="chasis_link"/>
         </joint>
     <joint name="arm_left_front_joint" type="fixed">
-        <origin xyz="-0.15 -0.0955 0.1" rpy="0.0 0.0 -1.5708"/>
+        <origin xyz="-0.15 -0.0955 0" rpy="0.0 0.0 -1.5708"/>
         <parent link="chasis_link"/>
         <child link="arm_left_front_link"/>
     </joint>
     <joint name="arm_left_back_joint" type="fixed">
-        <origin xyz="0.17 -0.0955 0.1" rpy="3.14 0.0 -1.5708"/>
+        <origin xyz="0.17 -0.0955 0.0" rpy="3.14 0.0 -1.5708"/>
         <parent link="chasis_link"/>
         <child link="arm_left_back_link"/>
     </joint>
     <joint name="arm_right_front_joint" type="fixed">
-        <origin xyz="-0.15 0.0955 0.1" rpy="0.0 3.14  -1.5708"/>
+        <origin xyz="-0.15 0.0955 0.0" rpy="0.0 3.14  -1.5708"/>
         <parent link="chasis_link"/>
         <child link="arm_right_front_link"/>
     </joint>
     <joint name="arm_right_back_joint" type="fixed">
-        <origin xyz="0.17 0.0955 0.1" rpy="3.14 3.14  -1.5708"/>
+        <origin xyz="0.17 0.0955 0.0" rpy="3.14 3.14  -1.5708"/>
         <parent link="chasis_link"/>
         <child link="arm_right_back_link"/>
@@ -201,5 +201,5 @@
     <!--Wheel Joints Definition-->
     <joint name="wheel_left_front_joint" type="continuous">
-        <origin xyz="${0.03+length_wheel/2} -0.067 -0.04 " rpy="3.14 -1.5708 0.0"/>
+        <origin xyz="${0.03+length_wheel/2} -0.067 -0.04 " rpy="0 ${pi/2} 0.0"/>
         <parent link="arm_left_front_link"/>
         <child link="wheel_left_front_link"/>
@@ -207,5 +207,5 @@
     </joint>
     <joint name="wheel_left_back_joint" type="continuous">
-        <origin xyz="${0.03+length_wheel/2} -0.067 0.04 " rpy="3.14 -1.5708 0.0"/>
+        <origin xyz="${0.03+length_wheel/2} -0.067 0.04 " rpy="0 ${pi/2} 0.0"/>
         <parent link="arm_left_back_link"/>
         <child link="wheel_left_back_link"/>
@@ -213,5 +213,5 @@
     </joint>
     <joint name="wheel_right_front_joint" type="continuous">
-        <origin xyz="${0.03+length_wheel/2} -0.067 0.04 " rpy="3.14 -1.5708 0.0"/>
+        <origin xyz="${0.03+length_wheel/2} -0.067 0.04 " rpy="0 -${pi/2} 0.0"/>
         <parent link="arm_right_front_link"/>
         <child link="wheel_right_front_link"/>
@@ -219,5 +219,5 @@
     </joint>
     <joint name="wheel_right_back_joint" type="continuous">
-        <origin xyz="${0.03+length_wheel/2} -0.067 -0.04 " rpy="3.14 -1.5708 0.0"/>
+        <origin xyz="${0.03+length_wheel/2} -0.067 -0.04 " rpy="0.0 -${pi/2} 0.0"/>
         <parent link="arm_right_back_link"/>
         <child link="wheel_right_back_link"/>

File: description/wheel.xacro (robot description, xacro)
@@ -1,4 +1,4 @@
 <?xml version="1.0"?>
-<robot xmlns:xacro="http://www.ros.org/wiki/xacro"  name="robot">
+<robot xmlns:xacro="http://www.ros.org/wiki/xacro"  name="rover">
     <xacro:property name="length_wheel" value="0.04"/>
     <xacro:property name="radius_wheel" value="0.07"/>

Commit message: Change dir of rover

File: description/gazebo.xacro (robot description, xacro)
@@ -11,18 +11,18 @@
         </ros>
         <!-- Update rate -->
-        <update_rate>500</update_rate>
+        <update_rate>100</update_rate>
         <!-- Number of wheel pairs -->
         <num_wheel_pairs>2</num_wheel_pairs>
+        <!-- wheels1-->
+        <right_joint>wheel_left_back_joint</right_joint>
+        <left_joint>wheel_right_back_joint</left_joint>
         <!-- wheels0 -->
-        <left_joint>wheel_left_front_joint</left_joint>
-        <right_joint>wheel_right_front_joint</right_joint>
-        <!-- wheels1-->
-        <left_joint>wheel_left_back_joint</left_joint>
-        <right_joint>wheel_right_back_joint</right_joint>
+        <right_joint>wheel_left_front_joint</right_joint>
+        <left_joint>wheel_right_front_joint</left_joint>
         <!-- kinematics -->
         <wheel_separation>0.4</wheel_separation>
         <wheel_separation>0.4</wheel_separation>
-        <wheel_diameter>0.14</wheel_diameter>
-        <wheel_diameter>0.14</wheel_diameter>
+        <wheel_diameter>0.15</wheel_diameter>
+        <wheel_diameter>0.15</wheel_diameter>
         <!-- limits -->
         <max_wheel_torque>400</max_wheel_torque>

File: description/lidar.xacro (robot description, xacro)
@@ -2,5 +2,5 @@
 <robot xmlns:xacro="http://www.ros.org/wiki/xacro"  name="rover">
     <joint name="laser_joint" type="fixed">
-        <origin xyz="0.075 0.0 0.085" rpy="0.0 0.0 0.0"/>
+        <origin xyz="-0.075 0.0 0.085" rpy="0.0 0.0 0.0"/>
         <parent link="chasis_link"/>
         <child link="laser_frame"/>

File: description/robot.xacro (robot description, xacro)
@@ -95,5 +95,5 @@
         </xacro:inertial_box>
         <visual>
-            <origin xyz="0.0 0.0115 -0.1" rpy="0.0 0.0 -1.5708"/>
+            <origin xyz="0.0 -0.01 -0.1" rpy="0.0 0.0 1.5708"/>
             <geometry>
                 <mesh filename="file://$(find rover)/description/stl/Chasis.stl" scale="0.01 0.01 0.01"/>
@@ -211,5 +211,5 @@
         <parent link="arm_left_front_link"/>
         <child link="wheel_left_front_link"/>
-        <axis xyz="0.0 0.0 1.0"/>
+        <axis xyz="0.0 0.0 -1.0"/>
     </joint>
     <joint name="wheel_left_back_joint" type="continuous">
@@ -217,5 +217,5 @@
         <parent link="arm_left_back_link"/>
         <child link="wheel_left_back_link"/>
-        <axis xyz="0.0 0.0 1.0"/>
+        <axis xyz="0.0 0.0 -1.0"/>
     </joint>
     <joint name="wheel_right_front_joint" type="continuous">
@@ -223,5 +223,5 @@
         <parent link="arm_right_front_link"/>
         <child link="wheel_right_front_link"/>
-        <axis xyz="0.0 0.0 1.0"/>
+        <axis xyz="0.0 0.0 -1.0"/>
     </joint>
     <joint name="wheel_right_back_joint" type="continuous">
@@ -229,5 +229,5 @@
         <parent link="arm_right_back_link"/>
         <child link="wheel_right_back_link"/>
-        <axis xyz="0.0 0.0 1.0"/>
+        <axis xyz="0.0 0.0 -1.0"/>
     </joint>
     <!--Link Definition-->
